Commit message: Alterado os arquivos URDF

File: ArmAgeddonRobot/urdf/hand.xacro (robot description, xacro)
@@ -12,10 +12,10 @@
       <visual>
         <geometry>
-          <mesh filename="package://franka_description/meshes/visual/hand.dae"/>
+          <mesh filename="package://ArmAgeddonRobot/meshes/visual/hand.dae"/>
         </geometry>
       </visual>
       <collision>
         <geometry>
-          <mesh filename="package://franka_description/meshes/collision/hand.stl"/>
+          <mesh filename="package://ArmAgeddonRobot/meshes/collision/hand.stl"/>
         </geometry>
       </collision>
@@ -24,10 +24,10 @@
       <visual>
         <geometry>
-          <mesh filename="package://franka_description/meshes/visual/finger.dae"/>
+          <mesh filename="package://ArmAgeddonRobot/meshes/visual/finger.dae"/>
         </geometry>
       </visual>
       <collision>
         <geometry>
-          <mesh filename="package://franka_description/meshes/collision/finger.stl"/>
+          <mesh filename="package://ArmAgeddonRobot/meshes/collision/finger.stl"/>
         </geometry>
       </collision>
@@ -37,5 +37,5 @@
         <origin xyz="0 0 0" rpy="0 0 ${pi}"/>
         <geometry>
-          <mesh filename="package://franka_description/meshes/visual/finger.dae"/>
+          <mesh filename="package://ArmAgeddonRobot/meshes/visual/finger.dae"/>
         </geometry>
       </visual>
@@ -43,5 +43,5 @@
         <origin xyz="0 0 0" rpy="0 0 ${pi}"/>
         <geometry>
-          <mesh filename="package://franka_description/meshes/collision/finger.stl"/>
+          <mesh filename="package://ArmAgeddonRobot/meshes/collision/finger.stl"/>
         </geometry>
       </collision>

File: ArmAgeddonRobot/urdf/panda_arm.urdf.xacro (robot description, xacro)
@@ -1,5 +1,5 @@
 <?xml version='1.0' encoding='utf-8'?>
 <robot xmlns:xacro="http://www.ros.org/wiki/xacro" name="panda">
-  <xacro:include filename="$(find franka_description)/robots/panda_arm.xacro" />
+  <xacro:include filename="$(find ArmAgeddonRobot)/urdf/panda_arm.xacro" />
   <xacro:panda_arm />
 </robot>

File: ArmAgeddonRobot/urdf/panda_arm.xacro (robot description, xacro)
@@ -1,5 +1,5 @@
 <?xml version='1.0' encoding='utf-8'?>
 <robot xmlns:xacro="http://www.ros.org/wiki/xacro" name="panda">
-  <xacro:macro name="panda_arm" params="arm_id:='panda' description_pkg:='franka_description' connected_to:='' xyz:='0 0 0' rpy:='0 0 0'">
+  <xacro:macro name="panda_arm" params="arm_id:='panda' description_pkg:='ArmAgeddonRobot' connected_to:='' xyz:='0 0 0' rpy:='0 0 0'">
     <xacro:unless value="${not connected_to}">
       <joint name="${arm_id}_joint_${connected_to}" type="fixed">

File: ArmAgeddonRobot/urdf/panda_arm_hand.urdf.xacro (robot description, xacro)
@@ -1,6 +1,6 @@
 <?xml version="1.0" encoding="utf-8"?>
 <robot xmlns:xacro="http://www.ros.org/wiki/xacro" name="panda">
-  <xacro:include filename="$(find franka_description)/robots/panda_arm.xacro"/>
-  <xacro:include filename="$(find franka_description)/robots/hand.xacro"/>
+  <xacro:include filename="$(find ArmAgeddonRobot)/urdf/panda_arm.xacro"/>
+  <xacro:include filename="$(find ArmAgeddonRobot)/urdf/hand.xacro"/>
   <xacro:panda_arm />
   <xacro:hand ns="panda" rpy="0 0 ${-pi/4}" connected_to="panda_link8"/>
