Commit message: OpenSCAD modelos
criado os modelos OpenSCAD
(URDF - não alterado)

File: ArmAgeddonRobot/urdf/robot.urdf (robot description, URDF)
Before this commit: robot ArmAgeddon, 10 links, 9 joints
Links:
- link base_1: geometry collision mesh filename=package://ArmAgeddonRobot/urdf/visual/base.stl; visual mesh filename=package://ArmAgeddonRobot/urdf/visual/base.stl
- link cubo_1: geometry collision mesh filename=package://ArmAgeddonRobot/urdf/visual/cubo.stl; visual mesh filename=package://ArmAgeddonRobot/urdf/visual/cubo.stl
- link flange_1: geometry collision mesh filename=package://ArmAgeddonRobot/urdf/visual/flange.stl; visual mesh filename=package://ArmAgeddonRobot/urdf/visual/flange.stl
- link link1_1: geometry collision mesh filename=package://ArmAgeddonRobot/urdf/visual/link1.stl; visual mesh filename=package://ArmAgeddonRobot/urdf/visual/link1.stl
- link link2_1: geometry collision mesh filename=package://ArmAgeddonRobot/urdf/visual/link2.stl; visual mesh filename=package://ArmAgeddonRobot/urdf/visual/link2.stl
- link link3_1: geometry collision mesh filename=package://ArmAgeddonRobot/urdf/visual/link3.stl; visual mesh filename=package://ArmAgeddonRobot/urdf/visual/link3.stl
- link link4_1: geometry collision mesh filename=package://ArmAgeddonRobot/urdf/visual/link4.stl; visual mesh filename=package://ArmAgeddonRobot/urdf/visual/link4.stl
- link link5_1: geometry collision mesh filename=package://ArmAgeddonRobot/urdf/visual/link5.stl; visual mesh filename=package://ArmAgeddonRobot/urdf/visual/link5.stl
- link welding_torch_1: geometry collision mesh filename=package://ArmAgeddonRobot/urdf/visual/welding_torch.stl; visual mesh filename=package://ArmAgeddonRobot/urdf/visual/welding_torch.stl

Commit message: UR10 - DEFINITIVO
#Ajustes no URDF
+ {Alterado} juntas do tcp e cubo para "fixed"
+ {Adicionado} os novos modelos de colisão
+ {Adicionado} a escala 0.001 aos modelos
+ {Removido} a colisão do cubo

File: ArmAgeddonRobot/urdf/robot.urdf (robot description, URDF)
Before this commit: robot ArmAgeddon, 10 links, 9 joints
Links:
- link base_1: geometry collision mesh filename=package://ArmAgeddonRobot/urdf/collision/base.stl scale=0.001 0.001 0.001; visual mesh filename=package://ArmAgeddonRobot/urdf/visual/base.stl
- link cubo_1: geometry visual mesh filename=package://ArmAgeddonRobot/urdf/visual/cubo.stl
- link flange_1: geometry collision mesh filename=package://ArmAgeddonRobot/urdf/collision/flange.stl scale=0.001 0.001 0.001; visual mesh filename=package://ArmAgeddonRobot/urdf/visual/flange.stl
- link link1_1: geometry collision mesh filename=package://ArmAgeddonRobot/urdf/collision/link1.stl scale=0.001 0.001 0.001; visual mesh filename=package://ArmAgeddonRobot/urdf/visual/link1.stl
- link link2_1: geometry collision mesh filename=package://ArmAgeddonRobot/urdf/collision/link2.stl scale=0.001 0.001 0.001; visual mesh filename=package://ArmAgeddonRobot/urdf/visual/link2.stl
- link link3_1: geometry collision mesh filename=package://ArmAgeddonRobot/urdf/collision/link3.stl scale=0.001 0.001 0.001; visual mesh filename=package://ArmAgeddonRobot/urdf/visual/link3.stl
- link link4_1: geometry collision mesh filename=package://ArmAgeddonRobot/urdf/collision/link4.stl scale=0.001 0.001 0.001; visual mesh filename=package://ArmAgeddonRobot/urdf/visual/link4.stl
- link link5_1: geometry collision mesh filename=package://ArmAgeddonRobot/urdf/collision/link5.stl scale=0.001 0.001 0.001; visual mesh filename=package://ArmAgeddonRobot/urdf/visual/link5.stl
- link welding_torch_1: geometry collision mesh filename=package://ArmAgeddonRobot/urdf/collision/welding_torch.stl scale=0.001 0.001 0.001; visual mesh filename=package://ArmAgeddonRobot/urdf/visual/welding_torch.stl
Joints:
- joint flange: axis 0 1 0 -> (none); limit lower=-6.28319 upper=6.28319 effort=1 velocity=20 -> (none); type revolute -> fixed
- joint tcp: axis 0 0 1 -> (none); limit lower=-6.28319 upper=6.28319 effort=1 velocity=20 -> (none); type revolute -> fixed

Commit message: rotação do TCP
Rotacionado o TCP para o padrão do Universal Robot

File: ArmAgeddonRobot/urdf/robot.urdf (robot description, URDF)
Before this commit: robot ArmAgeddon, 10 links, 9 joints
Links:
- link cubo_1: mass 0.766908 -> None; geometry 
Joints:
- joint tcp: origin xyz=0.00106366 -0.430726 0.00599082 rpy=0.677166 0.00744708 -3.13561 -> xyz=0.00106366 -0.430726 0.00599082 rpy=2.46443 -0.00744708 0.00598722

Commit message: Movido o TCP para o ponto de atuação
Movido o TCP para o ponto de atuação

File: ArmAgeddonRobot/urdf/robot.urdf (robot description, URDF)
Before this commit: robot ArmAgeddon, 10 links, 9 joints
Links:
- removed link cubo_1
- added link grasping_frame
Joints:
- removed joint tcp
- added joint grasping_frame_joint: type fixed, parent welding_torch_1, child grasping_frame, origin xyz=0.00106366 -0.430726 0.00599082 rpy=2.46443 -0.00744708 0.00598722
